File: IMU/BNO080/PCB_design/devBoard/devBoard.brd (EAGLE design)
At the start: 70.6 x 49.8 mm, 46 parts, among them IC1 XMEGA16A4A, U1 BNO080, U3 LTC3630EMSE, U4 NAVSPARK_MININAVSPARK_MINI, Y1 ABS07

Commit message: AVR SPI exmpl, board designs
Parts:
- added U$1: (no value), logos:LOGO_KLEIN
- added U$2: (no value), logos:HVA_LOGO
- C12: value 100p -> 10p
- L2: value 100u -> 33u
- R5: value 150k -> 47k
Changed lines of the file:
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@@
 <drawing>
 <settings>
-<setting alwaysvectorfont="yes"/>
+<setting alwaysvectorfont="no"/>
 <setting verticaltext="up"/>
 </settings>
@@
 <attribute name="NAME" x="27.55" y="8.53" size="1" layer="25" font="vector" ratio="17" align="center"/>
 </element>
-<element name="C12" library="Capacitor" package="0805" value="100p" x="10.61" y="22.86" smashed="yes" rot="R90">
+<element name="C12" library="Capacitor" package="0805" value="10p" x="10.61" y="22.86" smashed="yes" rot="R90">
 <attribute name="NAME" x="9.04" y="22.86" size="1" layer="25" font="vector" ratio="17" rot="R90" align="center"/>
 </element>
@@
 <attribute name="VALUE" x="39.475" y="42.7749" size="0.8128" layer="27"/>
 </element>
-<element name="L2" library="Inductor" package="DR73/74" value="100u" x="18.23" y="19.05" smashed="yes" rot="R90">
+<element name="L2" library="Inductor" package="DR73/74" value="33u" x="18.23" y="19.05" smashed="yes" rot="R90">
 <attribute name="NAME" x="22.16" y="14.58" size="1" layer="25" font="vector" ratio="17" align="center"/>
 </element>
-<element name="R5" library="Resistor" package="0805" value="150k" x="13.15" y="22.86" smashed="yes" rot="R90">
+<element name="R5" library="Resistor" package="0805" value="47k" x="13.15" y="22.86" smashed="yes" rot="R90">
 <attribute name="NAME" x="14.88" y="23.86" size="1" layer="25" font="vector" ratio="17" rot="R90" align="center"/>
 </element>
@@
 <element name="POWER1" library="Phoenix-con" package="CON_3.81MM2_SIDE" value="CON_3.81MM2_SIDE" x="19.5" y="7.62" smashed="yes"/>
 <element name="POWER2" library="Phoenix-con" package="CON_3.81MM2_SIDE" value="CON_3.81MM2_SIDE" x="9.34" y="7.62" smashed="yes"/>
+<element name="U$1" library="logos" package="LOGO_KLEIN" value="" x="51.6" y="11.9" smashed="yes" rot="MR0"/>
+<element name="U$2" library="logos" package="HVA_LOGO" value="" x="66.7" y="29.4" smashed="yes" rot="MR0"/>
 </elements>
 <signals>
